Commit message: created a urdf and a launch file

File: ros2_ws/src/my_robot_description/urdf/my_sol/arm.urdf (robot description, URDF)
Before this commit: robot my_robot, 7 links, 6 joints
Links:
- added link tool_link
Joints:
- added joint hand_tool_joint: type fixed, parent hand_link, child tool_link, origin xyz=0 0 0.02 rpy=0 0 0
