Commit message: added gripper urdf file

File: ros2_ws/src/my_robot_description/urdf/common_properties.xacro (robot description, xacro)
@@ -7,3 +7,9 @@
         <color rgba="0 0 0.5 1" />
     </material>
+    <material name="dark_green">
+        <color rgba="0 0.4 0 1" />
+    </material>
+    <material name="light_green">
+        <color rgba="0 0.6 0 1" />
+    </material>
 </robot>

File: ros2_ws/src/my_robot_description/urdf/my_robot.urdf.xacro (robot description, xacro)
@@ -2,4 +2,10 @@
 <robot name="my_robot" xmlns:xacro="http://www.ros.org/wiki/xacro">
     <xacro:include filename="common_properties.xacro" />
-    <xacro:include filename="arm.xacro" />
+    <xacro:include filename="arm.xacro" />j
+    <xacro:include filename="gripper.xacro" />
+    <joint name="gripper_base_joint" type="fixed">
+        <parent link="tool_link" />
+        <child link="gripper_base_link" />
+        <origin xyz="0 0 0" rpy="0 0 0" />
+    </joint>
 </robot>
